File: DesignFiles/SHV_Feedthrough_PulserPCB/SHV_Feedthrough_PulserPCB.kicad_pcb (KiCad board)
At the start: 2 copper layers, 17.7 x 17.7 mm, 13 parts, among them J1 CenterHole, J2 PulseLine, J3 PulseLine, J4 PulseLine, J5 PulseLine, J6 PulseLine, J7 PulseLine

Commit message: Added slots to pulser board. Updated instructions for cleaning.
Other:
- board text added: "V3"
- board text removed: "SHVFilter PulserBoard"
- board text removed: "V2"
Changed lines of the file:
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@@
       (effects (font (size 1 1) (thickness 0.15)))
     )
+    (fp_line (start 3.85812 -1.59809) (end 5.70588 -2.36345) (layer "Edge.Cuts") (width 0.12))
+    (fp_line (start 3.85812 1.59809) (end 5.70588 2.36345) (layer "Edge.Cuts") (width 0.12))
+    (fp_arc (start 5.70588 -2.36345) (mid 6.175999 0) (end 5.70588 2.36345) (layer "Edge.Cuts") (width 0.12))
+    (fp_arc (start 3.85812 -1.59809) (mid 4.176 0) (end 3.85812 1.59809) (layer "Edge.Cuts") (width 0.12))
     (pad "1" smd roundrect (at 2.632 0 300) (size 0.6 2.9) (layers "F.Cu" "F.Paste" "F.Mask") (roundrect_rratio 0.25)
       (net 1 "Net-(C1-Pad1)") (pintype "passive"))
@@
       (effects (font (size 1 1) (thickness 0.15)))
     )
+    (fp_line (start 3.85812 1.59809) (end 5.70588 2.36345) (layer "Edge.Cuts") (width 0.12))
+    (fp_line (start 3.85812 -1.59809) (end 5.70588 -2.36345) (layer "Edge.Cuts") (width 0.12))
+    (fp_arc (start 3.85812 -1.59809) (mid 4.176 0) (end 3.85812 1.59809) (layer "Edge.Cuts") (width 0.12))
+    (fp_arc (start 5.70588 -2.36345) (mid 6.175999 0) (end 5.70588 2.36345) (layer "Edge.Cuts") (width 0.12))
     (pad "1" smd roundrect (at 2.632 0 240) (size 0.6 2.9) (layers "F.Cu" "F.Paste" "F.Mask") (roundrect_rratio 0.25)
       (net 1 "Net-(C1-Pad1)") (pintype "passive"))
@@
   )
   (footprint "Library:HV2225SideMount" (layer "F.Cu")
-    (at 154 76 60)
+    (at 153.999997 76 60)
     (property "Sheetfile" "SHV_Feedthrough_PulserPCB.kicad_sch")
     (property "Sheetname" "")
@@
       (effects (font (size 1 1) (thickness 0.15)))
     )
+    (fp_line (start 3.85812 -1.59809) (end 5.70588 -2.36345) (layer "Edge.Cuts") (width 0.12))
+    (fp_line (start 3.85812 1.59809) (end 5.70588 2.36345) (layer "Edge.Cuts") (width 0.12))
+    (fp_arc (start 3.85812 -1.59809) (mid 4.176 0) (end 3.85812 1.59809) (layer "Edge.Cuts") (width 0.12))
+    (fp_arc (start 5.70588 -2.36345) (mid 6.175999 0) (end 5.70588 2.36345) (layer "Edge.Cuts") (width 0.12))
     (pad "1" smd roundrect (at 2.632 0 60) (size 0.6 2.9) (layers "F.Cu" "F.Paste" "F.Mask") (roundrect_rratio 0.25)
       (net 1 "Net-(C1-Pad1)") (pintype "passive"))
@@
       (effects (font (size 1 1) (thickness 0.15)))
     )
+    (fp_line (start 3.85812 1.59809) (end 5.70588 2.36345) (layer "Edge.Cuts") (width 0.12))
+    (fp_line (start 3.85812 -1.59809) (end 5.70588 -2.36345) (layer "Edge.Cuts") (width 0.12))
+    (fp_arc (start 5.70588 -2.36345) (mid 6.175999 0) (end 5.70588 2.36345) (layer "Edge.Cuts") (width 0.12))
+    (fp_arc (start 3.85812 -1.59809) (mid 4.176 0) (end 3.85812 1.59809) (layer "Edge.Cuts") (width 0.12))
     (pad "1" smd roundrect (at 2.632 0 120) (size 0.6 2.9) (layers "F.Cu" "F.Paste" "F.Mask") (roundrect_rratio 0.25)
       (net 1 "Net-(C1-Pad1)") (pintype "passive"))
@@
       (effects (font (size 1 1) (thickness 0.15)))
     )
+    (fp_line (start 3.85812 -1.59809) (end 5.70588 -2.36345) (layer "Edge.Cuts") (width 0.12))
+    (fp_line (start 3.85812 1.59809) (end 5.70588 2.36345) (layer "Edge.Cuts") (width 0.12))
+    (fp_arc (start 3.85812 -1.59809) (mid 4.176 0) (end 3.85812 1.59809) (layer "Edge.Cuts") (width 0.12))
+    (fp_arc (start 5.70588 -2.36345) (mid 6.175999 0) (end 5.70588 2.36345) (layer "Edge.Cuts") (width 0.12))
     (pad "1" smd roundrect (at 2.632 0 180) (size 0.6 2.9) (layers "F.Cu" "F.Paste" "F.Mask") (roundrect_rratio 0.25)
       (net 1 "Net-(C1-Pad1)") (pintype "passive"))
@@
   )
   (footprint "Library:HV2225SideMount" (layer "F.Cu")
-    (at 154 76)
+    (at 153.999997 76)
     (property "Sheetfile" "SHV_Feedthrough_PulserPCB.kicad_sch")
     (property "Sheetname" "")
@@
       (effects (font (size 1 1) (thickness 0.15)))
     )
+    (fp_line (start 3.85812 -1.59809) (end 5.70588 -2.36345) (layer "Edge.Cuts") (width 0.12))
+    (fp_line (start 3.85812 1.59809) (end 5.70588 2.36345) (layer "Edge.Cuts") (width 0.12))
+    (fp_arc (start 5.70588 -2.36345) (mid 6.175999 0) (end 5.70588 2.36345) (layer "Edge.Cuts") (width 0.12))
+    (fp_arc (start 3.85812 -1.59809) (mid 4.176 0) (end 3.85812 1.59809) (layer "Edge.Cuts") (width 0.12))
     (pad "1" smd roundrect (at 2.632 0) (size 0.6 2.9) (layers "F.Cu" "F.Paste" "F.Mask") (roundrect_rratio 0.25)
       (net 1 "Net-(C1-Pad1)") (pintype "passive"))
@@
   (gr_circle (center 154 76) (end 161.8 76) (layer "B.Mask") (width 0.9) (fill none))
   (gr_circle (center 154 76) (end 162.85 76) (layer "Edge.Cuts") (width 0.2) (fill none))
-  (gr_text "V2" (at 154 81) (layer "B.SilkS")
+  (gr_text "V3" (at 153.999997 82.8) (layer "B.SilkS")
     (effects (font (size 1 1) (thickness 0.15)) (justify mirror))
   )
-  (gr_text "SHVFilter\nPulserBoard" (at 154 71) (layer "B.SilkS")
-    (effects (font (size 1 1) (thickness 0.15)) (justify mirror))
-  )
